Commit message: separated urdf xacro for links and plugins

File: urdf/sjtu_drone.gazebo.xacro (robot description, xacro)
@@ -1,23 +1,4 @@
 <?xml version="1.0" ?>
 <robot name="sjtu_drone">
-  <link name="base_link">
-    <inertial>
-      <mass value="1.477"/>
-      <origin rpy="0 0 0" xyz="0 0 0"/>
-      <inertia ixx="0.1152" ixy="0" ixz="0" iyy="0.1152" iyz="0" izz="0.218"/>
-    </inertial>
-    <collision name="sjtu_drone__collision">
-      <origin rpy="0 0 0" xyz="0   0   0.04"/>
-      <geometry>
-        <mesh filename="package://sjtu_drone/meshes/quadrotor_4.stl"/>
-      </geometry>
-    </collision>
-    <visual name="sjtu_drone__visual">
-      <origin rpy="0 0 0" xyz="0   0   0.04"/>
-      <geometry>
-        <mesh filename="package://sjtu_drone/meshes/quadrotor_4.dae"/>
-      </geometry>
-    </visual>
-  </link>
   <gazebo>
     <plugin name='simple_drone' filename='libplugin_drone.so'>
@@ -50,39 +31,36 @@
   </gazebo>
   <!-- Sensors -->
+  <gazebo reference="imu_link">
+    	<sensor name='sensor_imu' type='imu'>
+          <always_on>1</always_on>
+          <update_rate>100</update_rate>
+        </sensor>
+	<material>Gazebo/Grey</material>
+  </gazebo>
   <gazebo>
-    	<sensor name='sensor_imu' type='imu'>
-        <always_on> 1 </always_on>
-        <update_rate> 100 </update_rate>
-        <pose> 0 0 0 0 0 0 </pose>
-        <plugin name='ros_imu' filename='libplugin_ros_imu.so'>
-        </plugin>
+        <plugin name='ros_imu' filename='libgazebo_ros_imu.so'>
+        <alwaysOn>true</alwaysOn>
+        <bodyName>imu_link</bodyName>
+        <frameName>imu_link</frameName>
+        <topicName>imu</topicName>
+        <serviceName>imu_service</serviceName>
+        <gaussianNoise>0.0</gaussianNoise>
+        <updateRate>0</updateRate>
         <imu>
           <noise>
-              <type>gaussian</type>
+            <type>gaussian</type>
             <rate>
-              <mean> 0 </mean>
-              <stddev> 0 </stddev>
+              <mean>0</mean>
+              <stddev>0</stddev>
             </rate>
             <accel>
-              <mean> 0 </mean>
-              <stddev> 0.00 </stddev>
+              <mean>0</mean>
+              <stddev>0.0</stddev>
             </accel>
           </noise>
         </imu>
-      </sensor>
-      <!-- Sonar sensor in 100fps -->
-      <sensor name='sensor_sonar' type='sonar'>
-        <always_on>1</always_on>
-        <visualize>0</visualize>
-        <update_rate>100</update_rate>
-        <pose> 0.5 0 0.3 0 1.570796327 3.141592653 </pose>
-        <plugin name='ros_sonar' filename='libplugin_ros_sonar.so'>
-        </plugin>
-        <sonar>
-          <min>0</min>
-          <max>5</max>
-          <radius>1.33974596</radius>
-        </sonar>
-      </sensor>
+      </plugin>
+  </gazebo>
+  <gazebo reference="camera_fwd_link">
     <!-- front camera -->
     <sensor name="front_camera" type="camera">
@@ -112,4 +90,6 @@
       </plugin>
     </sensor>
+  </gazebo>
+  <gazebo reference="camera_bot_link">
 	  <!-- downward looking camera -->
     <sensor name="down_camera" type="camera">
@@ -131,5 +111,4 @@
         </noise>
       </camera>
-      <pose> 0.0 0.0 0.0 0 1.570796326794897 0 </pose>
       <always_on>1</always_on>
       <update_rate>15</update_rate>
@@ -140,3 +119,19 @@
     </sensor>
   </gazebo>
+  <!-- gazebo reference="sonar_link">
+      <sensor name='sensor_sonar' type='sonar'>
+        <always_on>1</always_on>
+        <visualize>0</visualize>
+        <update_rate>100</update_rate>
+      </sensor>
+  </gazebo>
+  <gazebo>
+        <plugin name='ros_sonar' filename='libplugin_ros_sonar.so'>
+        </plugin>
+        <sonar>
+          <min>0</min>
+          <max>5</max>
+          <radius>1.33974596</radius>
+        </sonar>
+  </gazebo -->
 </robot>
